Commit message: Added recognition script and fixed launch files

File: robot_description/urdf/robot.urdf (robot description, URDF)
Before this commit: robot visual, 11 links, 10 joints
Links:
- removed link box
- removed link head
- removed link left_back_wheel
- removed link left_base
- removed link left_front_wheel
- removed link left_leg
- removed link right_back_wheel
- removed link right_base
- removed link right_front_wheel
- removed link right_leg
- added link base_footprint
- added link camera_link; visual cylinder length=0.05 radius=0.05
- added link front_caster; collision sphere radius=${(wheel_radius+wheel_zoff-(base_height/2))}; visual sphere radius=${(wheel_radius+wheel_zoff-(base_height/2))}
- link base_link: geometry collision box size=${base_length} ${base_width} ${base_height}; visual box size=${base_length} ${base_width} ${base_height}
Joints:
- removed joint base_to_left_leg
- removed joint base_to_right_leg
- removed joint head_swivel
- removed joint left_back_wheel_joint
- removed joint left_base_joint
- removed joint left_front_wheel_joint
- removed joint right_back_wheel_joint
- removed joint right_base_joint
- removed joint right_front_wheel_joint
- removed joint tobox
- added joint base_joint: type fixed, parent base_footprint, child base_link, origin xyz=0.0 0.0 ${(wheel_radius+wheel_zoff)} rpy=0 0 0
- added joint camera_joint: type fixed, parent base_link, child camera_link, origin xyz=${base_length/2} 0 ${base_height/2} rpy=0 0 0
- added joint caster_joint: type fixed, parent base_link, child front_caster, origin xyz=${caster_xoff} 0.0 ${-(base_height/2)} rpy=0 0 0
